File: sch/main_board.brd (EAGLE design)
At the start: 99.2 x 65.2 mm, 17 parts, among them IC1 MCP73831T-2ACI_OT

Commit message: Main board ver. 1.0
Parts:
- added JP1, JP2: (no value), pinhead-2:1X04SMD
- added R5: 10k, resistor:R1206
- added S1: (no value), switch:255SB
- added U$5: (no value), SamacSys_Parts:SOIC127P600X175-14N
- R4: value 316k -> 402k
- moved U$1 38.7 mm to (55.9, 10.2)
- moved R4 24.4 mm to (17.1, 34.4), turned to 180 degrees
- moved L1 21.2 mm to (21.6, 32.8), turned to 90 degrees
- moved U$4 21.0 mm to (80.0, 26.7), turned to 90 degrees
- moved R1 20.2 mm to (17.1, 31.4), turned to 0 degrees
- moved C4 16.2 mm to (16.9, 27.7), turned to 180 degrees
- moved U$2 16.0 mm to (21.6, 29.1), turned to 270 degrees
- moved R3 13.4 mm to (19.1, 12.2), turned to 180 degrees
- moved C5 12.0 mm to (25.4, 33.0), turned to 270 degrees
- moved D2 11.4 mm to (21.6, 24.1), turned to 0 degrees
- moved C1 10.9 mm to (27.9, 33.0), turned to 270 degrees
- moved LED1 9.25 mm to (22.9, 14.0), turned to 0 degrees
- moved R2 8.74 mm to (19.1, 14.9), turned to 0 degrees
- moved C3 8.07 mm to (17.7, 19.3), turned to 270 degrees
- moved C2 8.07 mm to (25.8, 19.3), turned to 270 degrees
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Connections:
- new net AD0/SDO: JP2.2, U$4.P$6, U$5.12
- new net BUFFER_EN: R5.1, U$3.28, U$5.1, U$5.13, U$5.4
- new net N$4: S1.1, U$1.P
- new net SCL/SCLK: JP1.1, U$4.P$3, U$5.3
- new net SDA/SDI: JP1.2, U$4.P$4, U$5.6
- net GND: now also JP1.4, U$5.10, U$5.7
- net MPU_INT: now also JP2.4; no longer U$4.P$5
- net SPI_CS_0: now also JP2.3
- net SPI_CS_1: now also U$4.P$7; no longer U$4.P$6
- net SPI_CS_2: now also U$4.P$8; no longer U$4.P$7
- net SPI_CS_3: now also U$4.P$9; no longer U$4.P$8
- net SPI_MISO: now also U$5.11; no longer U$4.P$9
- net SPI_MOSI: now also U$5.5; no longer U$4.P$4
- net SPI_SCK: now also U$5.2; no longer U$4.P$3
- net VCC: now also JP1.3, R5.2, U$4.P$5, U$5.14
- net V_BATT: now also S1.2; no longer U$1.P
Routing:
- net MPU_INT: track 0.00 -> 134.3 mm
- net VCC: track 0.00 -> 113.8 mm, vias 0 -> 5
- net SCL/SCLK: track 0.00 -> 110.1 mm
- net AD0/SDO: track 0.00 -> 109.4 mm
- net SDA/SDI: track 0.00 -> 98.3 mm
- net SPI_MISO: track 0.00 -> 61.0 mm
- net V_BATT: track 0.00 -> 57.8 mm
- net SPI_CS_0: track 0.00 -> 51.4 mm
- net BUFFER_EN: track 0.00 -> 49.7 mm
- net SPI_CS_3: track 0.00 -> 49.6 mm
- net SPI_MOSI: track 0.00 -> 46.0 mm
- net SPI_SCK: track 0.00 -> 40.6 mm
- net N$4: track 0.00 -> 25.1 mm, vias 1 -> 0
- net SPI_CS_1: track 0.00 -> 23.6 mm
- net SPI_CS_2: track 0.00 -> 20.8 mm
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- added copper zone on layer 16, net GND
- added copper zone on layer 1, net VCC
- added copper zone on layer 16, net VCC
Other:
- board size 99.2 x 65.2 mm -> 86.5 x 65.2 mm
- board text added: "!CS"
- board text added: "AD0 SDO"
- board text added: "BATT"
- board text added: "GND"
- board text added: "INT"
- board text added: "Praca Magisterska AGH, Elektronika i Telekomunikacja, Systemy Wbudowane Autor: Damian Świerk 2019"
- board text added: "SCL"
- board text added: "SDA"
- board text added: "VDD"
- board text added: "VDDIO"

Commit message: Ready for production HW version
Parts:
- R3: value 100 -> 150
- S1: value (none) -> 09.03201.02; device switch:255SB -> SamacSys_Parts:090320102
- turned S1 to 270 degrees
Connections:
- net N$4: now also S1.3; no longer S1.1
Routing:
- net V_BATT: track 57.8 -> 54.6 mm
- net N$4: track 25.1 -> 24.1 mm
Other:
- board text added: "1"
- board text added: "2"
- board text added: "3"
Changed lines of the file:
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@@
 <drawing>
 <settings>
-<setting alwaysvectorfont="yes"/>
+<setting alwaysvectorfont="no"/>
 <setting verticaltext="up"/>
 </settings>
@@
 <layer number="14" name="Route14" color="22" fill="1" visible="no" active="no"/>
 <layer number="15" name="Route15" color="23" fill="1" visible="no" active="no"/>
-<layer number="16" name="Bottom" color="1" fill="1" visible="no" active="yes"/>
+<layer number="16" name="Bottom" color="1" fill="1" visible="yes" active="yes"/>
 <layer number="17" name="Pads" color="2" fill="1" visible="yes" active="yes"/>
 <layer number="18" name="Vias" color="2" fill="1" visible="yes" active="yes"/>
@@
 <layer number="20" name="Dimension" color="24" fill="1" visible="yes" active="yes"/>
 <layer number="21" name="tPlace" color="7" fill="1" visible="yes" active="yes"/>
-<layer number="22" name="bPlace" color="7" fill="1" visible="no" active="yes"/>
+<layer number="22" name="bPlace" color="7" fill="1" visible="yes" active="yes"/>
 <layer number="23" name="tOrigins" color="15" fill="1" visible="yes" active="yes"/>
-<layer number="24" name="bOrigins" color="15" fill="1" visible="no" active="yes"/>
+<layer number="24" name="bOrigins" color="15" fill="1" visible="yes" active="yes"/>
 <layer number="25" name="tNames" color="7" fill="1" visible="yes" active="yes"/>
-<layer number="26" name="bNames" color="7" fill="1" visible="no" active="yes"/>
+<layer number="26" name="bNames" color="7" fill="1" visible="yes" active="yes"/>
 <layer number="27" name="tValues" color="7" fill="1" visible="no" active="yes"/>
 <layer number="28" name="bValues" color="7" fill="1" visible="no" active="yes"/>
@@
 <layer number="38" name="bTest" color="7" fill="1" visible="no" active="yes"/>
 <layer number="39" name="tKeepout" color="4" fill="11" visible="yes" active="yes"/>
-<layer number="40" name="bKeepout" color="1" fill="11" visible="no" active="yes"/>
+<layer number="40" name="bKeepout" color="1" fill="11" visible="yes" active="yes"/>
 <layer number="41" name="tRestrict" color="4" fill="10" visible="yes" active="yes"/>
-<layer number="42" name="bRestrict" color="1" fill="10" visible="no" active="yes"/>
+<layer number="42" name="bRestrict" color="1" fill="10" visible="yes" active="yes"/>
 <layer number="43" name="vRestrict" color="2" fill="10" visible="no" active="yes"/>
 <layer number="44" name="Drills" color="7" fill="1" visible="no" active="yes"/>
@@
 <layer number="50" name="dxf" color="7" fill="1" visible="no" active="no"/>
 <layer number="51" name="tDocu" color="7" fill="1" visible="yes" active="yes"/>
-<layer number="52" name="bDocu" color="7" fill="1" visible="no" active="yes"/>
+<layer number="52" name="bDocu" color="7" fill="1" visible="yes" active="yes"/>
 <layer number="53" name="tGND_GNDA" color="7" fill="9" visible="no" active="no"/>
 <layer number="54" name="bGND_GNDA" color="1" fill="9" visible="no" active="no"/>
@@
 Autor: Damian Świerk
 2019</text>
+<text x="77.4954" y="13.6144" size="1.016" layer="21" rot="R90">1</text>
+<text x="77.4954" y="10.9982" size="1.016" layer="21" rot="R90">2</text>
+<text x="77.4954" y="8.4582" size="1.016" layer="21" rot="R90">3</text>
 </plain>
 <attributes>
@@
 <param name="checkFont" value="1"/>
 <param name="checkRestrict" value="1"/>
-<param name="checkStop" value="0"/>
-<param name="checkValues" value="0"/>
+<param name="checkStop" value="1"/>
+<param name="checkValues" value="1"/>
 <param name="checkNames" value="1"/>
 <param name="checkWireStubs" value="1"/>
@@
 <attribute name="MOUSER_PART_NUMBER" value="579-MCP73831T-2ACIOT" x="21.59" y="19.05" size="1.778" layer="27" rot="R180" display="off"/>
 <attribute name="MOUSER_PRICE-STOCK" value="https://www.mouser.com/Search/Refine.aspx?Keyword=579-MCP73831T-2ACIOT" x="21.59" y="19.05" size="1.778" layer="27" rot="R180" display="off"/>
-<attribute name="NAME" x="20.32" y="16.51" size="1.27" layer="25" rot="R180" align="center"/>
+<attribute name="NAME" x="20.32" y="16.51" size="0.762" layer="25" rot="R180" align="center"/>
 <attribute name="VALUE" x="21.59" y="21.59" size="1.27" layer="27" rot="R180" align="center"/>
 </element>
@@
 <attribute name="VALUE" x="25.4" y="12.7" size="1.27" layer="27" rot="R90"/>
 </element>
-<element name="R3" library="resistor" library_urn="urn:adsk.eagle:library:348" package="R1206" package3d_urn="urn:adsk.eagle:package:23540/2" value="100" x="19.05" y="12.192" smashed="yes" rot="R180">
+<element name="R3" library="resistor" library_urn="urn:adsk.eagle:library:348" package="R1206" package3d_urn="urn:adsk.eagle:package:23540/2" value="150" x="19.05" y="12.192" smashed="yes" rot="R180">
 <attribute name="NAME" x="15.0114" y="13.2588" size="1.27" layer="25" rot="R270"/>
 <attribute name="VALUE" x="20.32" y="14.732" size="1.27" layer="27" rot="R180"/>
@@
 <attribute name="VALUE" x="75.6666" y="36.195" size="1.27" layer="27"/>
 </element>
-<element name="S1" library="switch" library_urn="urn:adsk.eagle:library:380" package="255SB" package3d_urn="urn:adsk.eagle:package:27679/1" value="" x="80.01" y="11.43" smashed="yes" rot="R90">
-<attribute name="NAME" x="78.994" y="3.302" size="1.27" layer="25" ratio="10" rot="R90"/>
-<attribute name="VALUE" x="76.454" y="11.43" size="1.27" layer="27" ratio="10" rot="R90"/>
+<element name="S1" library="SamacSys_Parts" package="090320102" value="09.03201.02" x="80.01" y="11.43" smashed="yes" rot="R270">
+<attribute name="DESCRIPTION" value="2 Way Through Hole SIP Switch SPST" x="80.01" y="11.43" size="1.778" layer="27" rot="R270" display="off"/>
+<attribute name="HEIGHT" value="5mm" x="80.01" y="11.43" size="1.778" layer="27" rot="R270" display="off"/>
+<attribute name="MANUFACTURER_NAME" value="EOZ" x="80.01" y="11.43" size="1.778" layer="27" rot="R270" display="off"/>
+<attribute name="MANUFACTURER_PART_NUMBER" value="09.03201.02" x="80.01" y="11.43" size="1.778" layer="27" rot="R270" display="off"/>
+<attribute name="MOUSER_PART_NUMBER" value="" x="80.01" y="11.43" size="1.778" layer="27" rot="R270" display="off"/>
+<attribute name="MOUSER_PRICE-STOCK" value="" x="80.01" y="11.43" size="1.778" layer="27" rot="R270" display="off"/>
+<attribute name="NAME" x="78.6384" y="4.2418" size="1.27" layer="25" align="center"/>
+<attribute name="RS_PART_NUMBER" value="1156283P" x="80.01" y="11.43" size="1.778" layer="27" rot="R270" display="off"/>
+<attribute name="RS_PRICE-STOCK" value="http://uk.rs-online.com/web/p/products/1156283P" x="80.01" y="11.43" size="1.778" layer="27" rot="R270" display="off"/>
+<attribute name="VALUE" x="80.01" y="11.43" size="1.27" layer="27" rot="R270" align="center"/>
 </element>
 </elements>
@@
 <vertex x="0" y="0.127"/>
 </polygon>
-<via x="73.4822" y="9.7028" extent="1-16" drill="0.45" diameter="1.2"/>
+<via x="65.8622" y="4.6228" extent="1-16" drill="0.45" diameter="1.2"/>
 <contactref element="U$5" pad="7"/>
 <contactref element="U$3" pad="8"/>
@@
 </polygon>
 <contactref element="S1" pad="2"/>
-<wire x1="80.01" y1="11.43" x2="22.86" y2="20.32" width="1.27" layer="16"/>
+<wire x1="80.01" y1="11.43" x2="26.543" y2="22.733" width="1.27" layer="16"/>
 </signal>
 <signal name="N$1" class="1">
@@
 </signal>
 <signal name="N$4">
+<contactref element="S1" pad="3"/>
 <contactref element="U$1" pad="P"/>
-<contactref element="S1" pad="1"/>
-<wire x1="55.9744875" y1="7.62" x2="80.01" y2="7.62" width="1.27" layer="16"/>
-<wire x1="55.9744875" y1="7.62" x2="55.88" y2="8.66" width="1.27" layer="16"/>
+<wire x1="55.88" y1="8.66" x2="80.01" y2="8.89" width="1.27" layer="16"/>
 </signal>
 </signals>

Commit message: Change feedback resistors for DC/DC converter
Parts:
- R1: value 100k -> 51k
- R4: value 402k -> 230k
Changed lines of the file:
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@@
 <attribute name="VALUE" x="21.59" y="32.766" size="1.27" layer="27" rot="R90" align="center"/>
 </element>
-<element name="R1" library="resistor" library_urn="urn:adsk.eagle:library:348" package="R1206" package3d_urn="urn:adsk.eagle:package:23540/2" value="100k" x="17.145" y="31.369" smashed="yes">
+<element name="R1" library="resistor" library_urn="urn:adsk.eagle:library:348" package="R1206" package3d_urn="urn:adsk.eagle:package:23540/2" value="51k" x="17.145" y="31.369" smashed="yes">
 <attribute name="NAME" x="14.3002" y="30.3022" size="1.27" layer="25" rot="R90"/>
 <attribute name="VALUE" x="15.875" y="28.829" size="1.27" layer="27"/>
 </element>
-<element name="R4" library="resistor" library_urn="urn:adsk.eagle:library:348" package="R1206" package3d_urn="urn:adsk.eagle:package:23540/2" value="402k" x="17.145" y="34.417" smashed="yes" rot="R180">
+<element name="R4" library="resistor" library_urn="urn:adsk.eagle:library:348" package="R1206" package3d_urn="urn:adsk.eagle:package:23540/2" value="230k" x="17.145" y="34.417" smashed="yes" rot="R180">
 <attribute name="NAME" x="18.288" y="36.83" size="1.27" layer="25" rot="R180"/>
 <attribute name="VALUE" x="18.415" y="36.957" size="1.27" layer="27" rot="R180"/>
