File: sch/main_board.sch (EAGLE design)
At the start: 22 parts, among them IC1 MCP73831T-2ACI_OT

Commit message: Ready for production HW version
Parts:
- R3: value 100 -> 150
- S1: value (none) -> 09.03201.02; device switch:255SB -> SamacSys_Parts:09.03201.02
Connections:
- net N$4: now also S1.3; no longer S1.O
- net V_BATT: now also S1.2; no longer S1.P
Changed lines of the file:
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@@
 <part name="D2" library="SamacSys_Parts" deviceset="VS-10BQ015-M3_5BT" device=""/>
 <part name="LED1" library="led" library_urn="urn:adsk.eagle:library:259" deviceset="LED" device="CHIPLED_1206" package3d_urn="urn:adsk.eagle:package:15823/2" value="GREEN"/>
-<part name="R3" library="resistor" library_urn="urn:adsk.eagle:library:348" deviceset="R-EU_" device="R1206" package3d_urn="urn:adsk.eagle:package:23540/2" value="100"/>
+<part name="R3" library="resistor" library_urn="urn:adsk.eagle:library:348" deviceset="R-EU_" device="R1206" package3d_urn="urn:adsk.eagle:package:23540/2" value="150"/>
 <part name="C2" library="resistor" library_urn="urn:adsk.eagle:library:348" deviceset="C-EU" device="C1206" package3d_urn="urn:adsk.eagle:package:23618/2" value="4.7u"/>
 <part name="C3" library="resistor" library_urn="urn:adsk.eagle:library:348" deviceset="C-EU" device="C1206" package3d_urn="urn:adsk.eagle:package:23618/2" value="4.7u"/>
@@
 <part name="JP2" library="pinhead-2" deviceset="PINHD-1X04" device="_2.54-SMD"/>
 <part name="P+6" library="supply1" library_urn="urn:adsk.eagle:library:371" deviceset="VCC" device=""/>
-<part name="S1" library="switch" library_urn="urn:adsk.eagle:library:380" deviceset="255SB" device="" package3d_urn="urn:adsk.eagle:package:27679/1"/>
 <part name="GND10" library="supply1" library_urn="urn:adsk.eagle:library:371" deviceset="GND" device=""/>
+<part name="S1" library="SamacSys_Parts" deviceset="09.03201.02" device=""/>
 </parts>
 <sheets>
@@
 <wire x1="187.96" y1="124.46" x2="187.96" y2="180.34" width="0.1524" layer="97" style="longdash"/>
 <wire x1="187.96" y1="180.34" x2="78.74" y2="180.34" width="0.1524" layer="97" style="longdash"/>
-<text x="-7.62" y="167.64" size="1.778" layer="97">Battery supply</text>
-<wire x1="-22.86" y1="180.34" x2="-22.86" y2="121.92" width="0.1524" layer="97" style="longdash"/>
-<wire x1="-22.86" y1="121.92" x2="76.2" y2="121.92" width="0.1524" layer="97" style="longdash"/>
+<text x="-25.4" y="175.26" size="1.778" layer="97">Battery supply</text>
+<wire x1="-27.94" y1="180.34" x2="-27.94" y2="121.92" width="0.1524" layer="97" style="longdash"/>
+<wire x1="-27.94" y1="121.92" x2="76.2" y2="121.92" width="0.1524" layer="97" style="longdash"/>
 <wire x1="76.2" y1="121.92" x2="76.2" y2="180.34" width="0.1524" layer="97" style="longdash"/>
-<wire x1="76.2" y1="180.34" x2="-22.86" y2="180.34" width="0.1524" layer="97" style="longdash"/>
+<wire x1="76.2" y1="180.34" x2="-27.94" y2="180.34" width="0.1524" layer="97" style="longdash"/>
 <wire x1="71.12" y1="116.84" x2="71.12" y2="-2.54" width="0.1524" layer="97" style="longdash"/>
 <wire x1="71.12" y1="-2.54" x2="-22.86" y2="-2.54" width="0.1524" layer="97" style="longdash"/>
@@
 </plain>
 <instances>
-<instance part="U$1" gate="G$1" x="-15.24" y="144.78" smashed="yes"/>
+<instance part="U$1" gate="G$1" x="-20.32" y="144.78" smashed="yes"/>
 <instance part="IC1" gate="G$1" x="22.86" y="152.4" smashed="yes">
 <attribute name="NAME" x="46.99" y="160.02" size="1.778" layer="95" align="center-left"/>
@@
 <attribute name="VALUE" x="165.1" y="109.22" size="1.778" layer="96" rot="R90"/>
 </instance>
-<instance part="S1" gate="1" x="5.08" y="152.4" smashed="yes" rot="R90">
-<attribute name="NAME" x="6.985" y="146.05" size="1.778" layer="95" rot="R180"/>
-<attribute name="VALUE" x="1.905" y="148.59" size="1.778" layer="96" rot="R180"/>
-</instance>
 <instance part="GND10" gate="1" x="134.62" y="66.04" smashed="yes">
 <attribute name="VALUE" x="132.08" y="63.5" size="1.778" layer="96"/>
+</instance>
+<instance part="S1" gate="G$1" x="12.7" y="149.86" smashed="yes" rot="R180">
+<attribute name="NAME" x="7.62" y="145.796" size="1.778" layer="95" rot="R180" align="center-left"/>
+<attribute name="VALUE" x="8.89" y="157.48" size="1.778" layer="96" rot="R180" align="center-left"/>
 </instance>
 </instances>
@@
 <wire x1="12.7" y1="129.54" x2="12.7" y2="132.08" width="0.1524" layer="91"/>
 <wire x1="12.7" y1="132.08" x2="12.7" y2="142.24" width="0.1524" layer="91"/>
-<wire x1="12.7" y1="142.24" x2="-5.08" y2="142.24" width="0.1524" layer="91"/>
+<wire x1="12.7" y1="142.24" x2="-10.16" y2="142.24" width="0.1524" layer="91"/>
 <pinref part="IC1" gate="G$1" pin="VSS"/>
 <wire x1="22.86" y1="149.86" x2="20.32" y2="149.86" width="0.1524" layer="91"/>
@@
 <segment>
 <pinref part="IC1" gate="G$1" pin="VBAT"/>
-<label x="12.7" y="154.94" size="1.778" layer="95" rot="R90" xref="yes"/>
+<label x="17.78" y="165.1" size="1.778" layer="95" rot="R180" xref="yes"/>
 <wire x1="22.86" y1="147.32" x2="17.78" y2="147.32" width="0.1524" layer="91"/>
 <pinref part="D2" gate="G$1" pin="A"/>
 <wire x1="30.48" y1="175.26" x2="17.78" y2="175.26" width="0.1524" layer="91"/>
-<wire x1="17.78" y1="175.26" x2="17.78" y2="154.94" width="0.1524" layer="91"/>
+<wire x1="17.78" y1="175.26" x2="17.78" y2="152.4" width="0.1524" layer="91"/>
 <junction x="17.78" y="147.32"/>
 <pinref part="C2" gate="G$1" pin="1"/>
-<wire x1="17.78" y1="154.94" x2="17.78" y2="147.32" width="0.1524" layer="91"/>
+<wire x1="17.78" y1="152.4" x2="17.78" y2="147.32" width="0.1524" layer="91"/>
 <wire x1="17.78" y1="139.7" x2="17.78" y2="147.32" width="0.1524" layer="91"/>
-<pinref part="S1" gate="1" pin="P"/>
-<wire x1="10.16" y1="154.94" x2="17.78" y2="154.94" width="0.1524" layer="91"/>
-<junction x="17.78" y="154.94"/>
+<pinref part="S1" gate="G$1" pin="2"/>
+<wire x1="12.7" y1="152.4" x2="17.78" y2="152.4" width="0.1524" layer="91"/>
+<junction x="17.78" y="152.4"/>
 </segment>
 </net>
@@
 <net name="N$4" class="0">
 <segment>
+<pinref part="S1" gate="G$1" pin="3"/>
+<wire x1="-7.62" y1="149.86" x2="-7.62" y2="147.32" width="0.1524" layer="91"/>
 <pinref part="U$1" gate="G$1" pin="+"/>
-<wire x1="-5.08" y1="147.32" x2="-2.54" y2="147.32" width="0.1524" layer="91"/>
-<pinref part="S1" gate="1" pin="O"/>
-<wire x1="-2.54" y1="147.32" x2="-2.54" y2="152.4" width="0.1524" layer="91"/>
-<wire x1="-2.54" y1="152.4" x2="0" y2="152.4" width="0.1524" layer="91"/>
+<wire x1="-7.62" y1="147.32" x2="-10.16" y2="147.32" width="0.1524" layer="91"/>
 </segment>
 </net>
@@
 </sheet>
 </sheets>
+<errors>
+</errors>
 </schematic>
 </drawing>

Commit message: Change feedback resistors for DC/DC converter
Parts:
- R1: value 100k -> 51k
- R4: value 402k -> 230k
Changed lines of the file:
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@@
 <part name="GND4" library="supply1" library_urn="urn:adsk.eagle:library:371" deviceset="GND" device=""/>
 <part name="L1" library="SamacSys_Parts" deviceset="SRN2512-2R2M" device=""/>
-<part name="R1" library="resistor" library_urn="urn:adsk.eagle:library:348" deviceset="R-EU_" device="R1206" package3d_urn="urn:adsk.eagle:package:23540/2" value="100k"/>
-<part name="R4" library="resistor" library_urn="urn:adsk.eagle:library:348" deviceset="R-EU_" device="R1206" package3d_urn="urn:adsk.eagle:package:23540/2" value="402k"/>
+<part name="R1" library="resistor" library_urn="urn:adsk.eagle:library:348" deviceset="R-EU_" device="R1206" package3d_urn="urn:adsk.eagle:package:23540/2" value="51k"/>
+<part name="R4" library="resistor" library_urn="urn:adsk.eagle:library:348" deviceset="R-EU_" device="R1206" package3d_urn="urn:adsk.eagle:package:23540/2" value="230k"/>
 <part name="GND3" library="supply1" library_urn="urn:adsk.eagle:library:371" deviceset="GND" device=""/>
 <part name="C4" library="resistor" library_urn="urn:adsk.eagle:library:348" deviceset="C-EU" device="C1206" package3d_urn="urn:adsk.eagle:package:23618/2" value="4.7u"/>

Commit message: Update schematic documentation
Other:
- note added: "Buffer and connector"
- note added: "Step-Down 5V - 3.3V"
- note removed: "Step-Down 5V - 3V"
Changed lines of the file:
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@@
 <sheet>
 <plain>
-<text x="83.82" y="175.26" size="1.778" layer="97">Step-Down 5V - 3V</text>
+<text x="83.82" y="175.26" size="1.778" layer="97">Step-Down 5V - 3.3V</text>
 <wire x1="78.74" y1="180.34" x2="78.74" y2="124.46" width="0.1524" layer="97" style="longdash"/>
 <wire x1="78.74" y1="124.46" x2="187.96" y2="124.46" width="0.1524" layer="97" style="longdash"/>
@@
 <wire x1="185.42" y1="116.84" x2="152.4" y2="116.84" width="0.1524" layer="97" style="longdash"/>
 <text x="153.416" y="114.3" size="1.778" layer="97">MPU-9250</text>
+<text x="119.38" y="111.76" size="1.9304" layer="97">Buffer and connector</text>
 </plain>
 <instances>
